File: Senior Design Power.kicad_sch (KiCad schematic)
At the start: 55 parts, among them J1 Screw_Terminal_01x03, J2 Screw_Terminal_01x04, J3 Screw_Terminal_01x04, Q1 Si7617DN, Q2 Si7617DN, Q3 SIS412DN, Q4 SIS412DN, U1 BQ24610

Commit message: updated to include EVM board components
Parts:
- removed CTTC1: 0.11u, Capacitor_SMD:C_0201_0603Metric, symbol Device:C
- removed D2, D3, D4: LED, LED_SMD:LED_0201_0603Metric, symbol Device:LED
- removed J2: Screw_Terminal_01x04, symbol Connector:Screw_Terminal_01x04
- removed R11, R12, R13: 10k, Resistor_SMD:R_0201_0603Metric, symbol Device:R
- added C21: 1.0uf, symbol Device:C
- added C22, C23: 0.1uf, symbol Device:C
- added C24: 2.2u, LED_SMD:LED_0201_0603Metric, symbol Device:C
- added C25: 0.1u, Capacitor_SMD:C_0201_0603Metric, symbol Device:C
- added Cff2: 22p, Capacitor_SMD:C_0201_0603Metric, symbol Device:C
- added D10, D5, D6, D7, D8, D9: LED, symbol Device:LED
- added J4: Screw_Terminal_01x04, symbol Connector:Screw_Terminal_01x04
- added JP1, JP3: Jumper_3_Open, symbol Jumper:Jumper_3_Open
- added JP2, JP4, JP5: Jumper_2_Open, symbol Jumper:Jumper_2_Open
- added Q5, Q6: TP0610L, Package_TO_SOT_THT:TO-92L_Inline, symbol Transistor_FET:TP0610L
- added Q7, Q8, Q9: 2N7002, Package_TO_SOT_SMD:SOT-23, symbol Transistor_FET:2N7002
- added R23, R25, R26, R4, R7: 100k, symbol Device:R
- added R24, R28, R29, R30, R31, R6: 2.21k, symbol Device:R
- added R27, R5: 10k, symbol Device:R
- added R32: 2, Resistor_SMD:R_0201_0603Metric, symbol Device:R
- added TP1: CHGEN, symbol Connector:TestPoint
- added TP10: ACDRV, symbol Connector:TestPoint
- added TP11: ACSET, symbol Connector:TestPoint
- added TP12: ISET1, symbol Connector:TestPoint
- added TP13: ISET2, symbol Connector:TestPoint
- added TP14: TS, symbol Connector:TestPoint
- added TP15: TTC, symbol Connector:TestPoint
- added TP16: TP13, symbol Connector:TestPoint
- added TP2: VCC, symbol Connector:TestPoint
- added TP3: GND, symbol Connector:TestPoint
- added TP4: VREF, symbol Connector:TestPoint
- added TP5: REGN, symbol Connector:TestPoint
- added TP6: PG, symbol Connector:TestPoint
- added TP7: STAT1, symbol Connector:TestPoint
- added TP8: STAT2, symbol Connector:TestPoint
- added TP9: BATDRV, symbol Connector:TestPoint
- C15: value C -> 0.1u
- C17: value C -> 0.1u; footprint (none) -> Resistor_SMD:R_0201_0603Metric
- C18, C19, C20: value C -> 0.1uf
- R15, R19, R8: value R -> 100k
- R21: value R -> 22.1k
- R22: value R -> 10k
- R3: value R -> 32.4k
Connections:
- net ACSET: now also TP11.1
- net Adapter +: now also R32.1
- net Battery Pack +: now also C17.1, C25.1
- net GND: now also C17.2, J1.2 (Pin_2), C21.1, C22.2, C23.1, C24.2, C25.2, Cff2.2, JP3.3 (B), Q7.2 (S), Q8.2 (S), Q9.2 (S), R23.2, R26.2, R4.2, TP3.1
- net ISET1: now also TP12.1
- net ISET2: now also TP13.1
- net VPULLUP: now also C23.2, JP1.2 (C), JP2.2 (B), JP3.1 (A)
- net VREF: now also J4.2 (Pin_2), JP1.3 (B), TP4.1; no longer U1.4 (CE)
- net V_PULLUP: now also JP4.2 (B)
- net at C2.1, C3.1, Q2.5 (D)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: now also C15.2
- net at C14.2, Q1.4 (G), Q2.4 (G)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: now also C15.1
- net at Cff1.2, R1.1, R2.2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: now also Cff2.1, TP16.1
- net STAT1: now reaches U1.5 (STAT1)
- net STAT1: now also D8.1 (K), TP7.1
- net TTC: now reaches U1.7 (TTC)
- net TTC: now also J1.1 (Pin_1), C22.1, JP3.2 (C), TP15.1
- net PG: now reaches U1.8 (~{PG})
- net PG: now also D7.1 (K), J4.4 (Pin_4), TP6.1
- net REGN: now reaches C5.1, D1.2, U1.17 (GND), U1.18 (REGN)
- net REGN: now also TP5.1
- net BATDRV: now reaches U1.23 (~{BATDRV})
- net BATDRV: now also R27.2, TP9.1
- net STAT2: now reaches U1.9 (STAT2)
- net STAT2: now also D9.1 (K), TP8.1
- net VEXT: now reaches J1.3 (Pin_3)
- net VEXT: now also C21.2, JP1.1 (A)
- new net: D10.2 (A), R28.2
- new net: Q6.1 (S), R25.1
- new net: Q6.2 (G), R27.1
- new net: JP5.1 (A), Q6.3 (D)
- new net: C24.1, R32.2
- new net: Q5.1 (S), R7.1
- new net: Q8.1 (G), R23.1, R7.2
- new net: Q7.1 (G), R25.2, R26.1
- new net: D6.1 (K), Q7.3 (D)
- new net: D9.2 (A), R31.2
- new net: D5.2 (A), R6.2
- new net: Q5.2 (G), R5.1
- new net: D10.1 (K), Q9.3 (D)
- new net: D5.1 (K), Q8.3 (D)
- new net: D8.2 (A), R30.2
- new net: D6.2 (A), R24.2
- new net: D7.2 (A), R29.2
- new net ACDRV: R5.2, TP10.1
- new net CHGEN: J4.3 (Pin_3), JP4.1 (A), Q9.1 (G), R4.1, TP1.1, U1.4 (CE)
- new net LEDPWR: JP2.1 (A), Q5.3 (D), R24.1, R28.1, R29.1, R30.1, R31.1, R6.1
- new net TS: J4.1 (Pin_1), TP14.1
- new net VCC: JP5.2 (B), TP2.1
Other:
- moved on the sheet: C16, C7, J1, R20

Commit message: PCB Review Day, Nov 17th - Ty
Parts:
- added C26: 1u, symbol Device:C
- added C27, C28: 10u, symbol Device:C
- added C29: 0.1u, symbol Device:C
- added D2: Zener - 1A, 40V, DIODE_SOD-523_DIO, symbol D1 Senior Design:ZLLS350TA
- added D9: BZX84C7V5, symbol Device:D_Zener
- added R11: 0, Resistor_SMD:R_0201_0603Metric, symbol Device:R
- added R12: 1k, symbol Device:R
- added R13, R33, R34, R36: 0, symbol Device:R
- added R35: 10, symbol Device:R
- C12, C13: value 20u -> 10u
- C25: value 0.1u -> 10u
- C5: footprint Capacitor_SMD:C_0201_0603Metric -> (none)
- L1: value 3.3u -> 4.7u
Connections:
- net Battery Pack +: now also R33.2, R34.2; no longer C11.2, C17.1, Cff1.1, R2.1, U1.13 (SRN)
- net CHGEN: now also R13.1; no longer U1.4 (CE)
- net GND: now also U1.17 (GND), C26.2, C27.1, C28.2, C29.2, D2.2
- net REGN: no longer U1.17 (GND)
- net System: now also C26.1, C27.2, C28.1, R11.1; no longer C3.2, C7.1, U1.1 (ACN), U1.24 (VCC)
- net at C6.1, L1.1, Q3.3 (S)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: now also D2.1
- net at C6.2, D1.1: now also R35.1; no longer U1.22 (BTST)
- net at U1.21 (HIDRV): now also R36.1; no longer Q3.2 (G)
- net at U1.3 (~{ACDRV}): now also D9.2 (A), R12.2; no longer R18.2
- new net: C29.1, C3.2, R11.2, U1.1 (ACN)
- new net: Q3.2 (G), R36.2
- new net: Cff1.1, R2.1, R34.1
- new net: R13.2, U1.4 (CE)
- new net: R12.1, R18.2
- new net: R35.2, U1.22 (BTST)
- new net: C11.2, C17.1, R33.1, U1.13 (SRN)
- new net PVCC: C7.1, D9.1 (K), U1.24 (VCC)
Other:
- moved on the sheet: C11, C25, C8
