File: Senior Design Power.kicad_sch (KiCad schematic)
At the start: 113 parts, among them J1 Screw_Terminal_01x03, J3 Screw_Terminal_01x04, J4 Screw_Terminal_01x04, Q1 Si7617DN, Q2 Si7617DN, Q3 SIS412DN, Q4 SIS412DN, Q5 TP0610L, Q6 TP0610L, Q7 2N7002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

Commit message: Nov 21st - Final Docs prior to order
Parts:
- removed C22: 0.1uf, symbol Device:C
- added CTTC1: 0.11, symbol Device:C
- Q5, Q6: value TP0610L -> TP0610K
- R10: value R -> 430k
- R19: value 100k -> 50k
- R21: value 22.1k -> 75k
- R22: value 10k -> 25k
- R9: value R -> 9.31k
- renumbered J1 to J2
Connections:
- net GND: now also CTTC1.2
- net LEDPWR: now also Q5.1 (S); no longer Q5.3 (D)
- net TTC: now also CTTC1.1
- net at Q6.1 (S): now also JP5.1 (A); no longer R25.1
- net at Q6.3 (D): now also R25.1; no longer JP5.1 (A)
- net at R7.1: now also Q5.3 (D); no longer Q5.1 (S)
Changed lines of the file:
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@@
 	)
 	(junction
+		(at 41.91 238.76)
+		(diameter 0)
+		(color 0 0 0 0)
+	)
+	(junction
 		(at 45.72 356.87)
 		(diameter 0)
@@
 	)
 	(junction
-		(at 41.91 238.76)
-		(diameter 0)
-		(color 0 0 0 0)
-	)
-	(junction
 		(at 34.29 55.88)
 		(diameter 0)
@@
 		(color 0 0 0 0)
 	)
+	(bus_entry
+		(at 189.23 30.48)
+		(size 2.54 2.54)
+		(stroke
+			(width 0)
+			(type default)
+		)
+	)
 	(wire
 		(pts
@@
 	(wire
 		(pts
+			(xy 41.91 238.76) (xy 50.8 238.76)
+		)
+		(stroke
+			(width 0)
+			(type default)
+		)
+	)
+	(wire
+		(pts
 			(xy 58.42 226.06) (xy 60.96 226.06)
 		)
@@
 	(wire
 		(pts
-			(xy 41.91 238.76) (xy 50.8 238.76)
+			(xy 31.75 238.76) (xy 41.91 238.76)
 		)
 		(stroke
@@
 	(wire
 		(pts
-			(xy 31.75 238.76) (xy 41.91 238.76)
-		)
-		(stroke
-			(width 0)
-			(type default)
-		)
-	)
-	(wire
-		(pts
 			(xy 144.78 232.41) (xy 144.78 224.79)
 		)
@@
 	)
 	(symbol
+		(lib_id "Device:C")
+		(at 41.91 242.57 0)
+		(unit 1)
+		(exclude_from_sim no)
+		(in_bom yes)
+		(on_board yes)
+		(dnp no)
+		(fields_autoplaced yes)
+		(property "Reference" "CTTC1"
+			(at 45.72 241.2999 0)
+			(effects
+				(font
+					(size 1.27 1.27)
+				)
+				(justify left)
+			)
+		)
+		(property "Value" "0.11"
+			(at 45.72 243.8399 0)
+			(effects
+				(font
+					(size 1.27 1.27)
+				)
+				(justify left)
+			)
+		)
+		(property "Footprint" ""
+			(at 42.8752 246.38 0)
+			(effects
+				(font
+					(size 1.27 1.27)
+				)
+				(hide yes)
+			)
+		)
+		(property "Datasheet" "~"
+			(at 41.91 242.57 0)
+			(effects
+				(font
+					(size 1.27 1.27)
+				)
+				(hide yes)
+			)
+		)
+		(property "Description" "Unpolarized capacitor"
+			(at 41.91 242.57 0)
+			(effects
+				(font
+					(size 1.27 1.27)
+				)
+				(hide yes)
+			)
+		)
+		(pin "2"
+		)
+		(pin "1"
+		)
+		(instances
+			(project ""
+				(path "/1b03766d-ecb9-4ef9-8b6d-907ca2bc5b89"
+					(reference "CTTC1")
+					(unit 1)
+				)
+			)
+		)
+	)
+	(symbol
 		(lib_id "Transistor_FET:Si7617DN")
 		(at 73.66 58.42 270)
@@
 		(lib_id "Transistor_FET:TP0610L")
 		(at 43.18 331.47 0)
+		(mirror x)
 		(unit 1)
 		(exclude_from_sim no)
@@
 		(on_board yes)
 		(dnp no)
-		(fields_autoplaced yes)
 		(property "Reference" "Q6"
-			(at 49.53 330.1999 0)
+			(at 49.53 332.7401 0)
 			(effects
 				(font
@@
 			)
 		)
-		(property "Value" "TP0610L"
-			(at 49.53 332.7399 0)
+		(property "Value" "TP0610K"
+			(at 49.53 330.2001 0)
 			(effects
 				(font
@@
 		)
 		(property "Footprint" "Package_TO_SOT_THT:TO-92L_Inline"
-			(at 48.26 333.375 0)
+			(at 48.26 329.565 0)
 			(effects
 				(font
@@
 		)
 		(property "Datasheet" "http://www.vishay.com/docs/70209/70209.pdf"
-			(at 48.26 335.28 0)
+			(at 48.26 327.66 0)
 			(effects
 				(font
@@
 			)
 		)
-		(property "Value" "100k"
+		(property "Value" "50k"
 			(at 76.2 270.5099 0)
 			(effects
@@
 			)
 		)
-		(property "Value" "R"
+		(property "Value" "430k"
 			(at 102.87 162.5599 0)
 			(effects
@@
 			)
 		)
-		(property "Value" "22.1k"
+		(property "Value" "75k"
 			(at 76.2 289.5599 0)
 			(effects
@@
 			)
 		)
-		(property "Value" "10k"
+		(property "Value" "25k"
 			(at 113.03 289.5599 0)
 			(effects
@@
 		(lib_id "Transistor_FET:TP0610L")
 		(at 12.7 331.47 0)
+		(mirror x)
 		(unit 1)
 		(exclude_from_sim no)
@@
 		(dnp no)
 		(property "Reference" "Q5"
-			(at 4.318 325.12 0)
+			(at 5.08 325.628 0)
 			(effects
 				(font
@@
 			)
 		)
-		(property "Value" "TP0610L"
-			(at 4.318 327.66 0)
+		(property "Value" "TP0610K"
+			(at 4.318 327.914 0)
 			(effects
 				(font
@@
 		)
 		(property "Footprint" "Package_TO_SOT_THT:TO-92L_Inline"
-			(at 17.78 333.375 0)
+			(at 17.78 329.565 0)
 			(effects
 				(font
@@
 		)
 		(property "Datasheet" "http://www.vishay.com/docs/70209/70209.pdf"
-			(at 17.78 335.28 0)
+			(at 17.78 327.66 0)
 			(effects
 				(font
@@
 	)
 	(symbol
-		(lib_id "Device:C")
-		(at 41.91 242.57 0)
-		(unit 1)
-		(exclude_from_sim no)
-		(in_bom yes)
-		(on_board yes)
-		(dnp no)
-		(fields_autoplaced yes)
-		(property "Reference" "C22"
-			(at 45.72 241.2999 0)
-			(effects
-				(font
-					(size 1.27 1.27)
-				)
-				(justify left)
-			)
-		)
-		(property "Value" "0.1uf"
-			(at 45.72 243.8399 0)
-			(effects
-				(font
-					(size 1.27 1.27)
-				)
-				(justify left)
-			)
-		)
-		(property "Footprint" ""
-			(at 42.8752 246.38 0)
-			(effects
-				(font
-					(size 1.27 1.27)
-				)
-				(hide yes)
-			)
-		)
-		(property "Datasheet" "~"
-			(at 41.91 242.57 0)
-			(effects
-				(font
-					(size 1.27 1.27)
-				)
-				(hide yes)
-			)
-		)
-		(property "Description" "Unpolarized capacitor"
-			(at 41.91 242.57 0)
-			(effects
-				(font
-					(size 1.27 1.27)
-				)
-				(hide yes)
-			)
-		)
-		(pin "2"
-		)
-		(pin "1"
-		)
-		(instances
-			(project "Senior Design Power"
-				(path "/1b03766d-ecb9-4ef9-8b6d-907ca2bc5b89"
-					(reference "C22")
-					(unit 1)
-				)
-			)
-		)
-	)
-	(symbol
 		(lib_id "Device:LED")
 		(at 138.43 339.09 90)
@@
 			)
 		)
-		(property "Value" "R"
+		(property "Value" "9.31k"
 			(at 102.87 148.5899 0)
 			(effects
@@
 		(dnp no)
 		(fields_autoplaced yes)
-		(property "Reference" "J1"
+		(property "Reference" "J2"
 			(at 26.67 220.98 0)
 			(effects
@@
 			(project ""
 				(path "/1b03766d-ecb9-4ef9-8b6d-907ca2bc5b89"
-					(reference "J1")
+					(reference "J2")
 					(unit 1)
 				)
